File: Project05-Circuit-Design-2/Project05-KiCad/Project05-KiCad.kicad_sch (KiCad schematic)
At the start: 4 parts

Commit message: Finish Project 5
Parts:
- added RL1: 30k, symbol Device:R
Connections:
- net GND: now also RL1.2
- net at C1.2, R1.2: now also RL1.1
Other:
- moved on the sheet: C1, R1, Rs1, Vs1
